Commit message: option for different cam distortion coefficient & DVL rangde aided feature depth estimation

File: config/GLRC/glrc.urdf (robot description, URDF)
Before this commit: robot rov, 7 links, 6 joints
Joints:
- removed joint right_cam_to_left_cam
- added joint ahrs_to_left_cam: type fixed, parent ahrs, child left_camera, origin xyz=0.310759 0.122349 -0.277866 rpy=-3.140161 -0.005635 1.562934
